Commit message: changed vfov of sonar  to 30 degrees

File: src/eca_a9/eca_a9_description/urdf/eca_a9_sensors.xacro (robot description, xacro)
@@ -118,5 +118,5 @@
       <origin xyz="0 0 0" rpy="0 0 0"/>
     </xacro:default_chemical_concentration_sensor>
-    <!--multibeam_blueview_p900_raster -->
+    <!--multibeam_blueview_p900_raster (working)-->
      <xacro:multibeam_blueview_p900_macro
       name="${namespace}"

File: src/nps_uw_multibeam_sonar/urdf/multibeam_sonar_blueview_p900.xacro (robot description, xacro)
@@ -22,5 +22,5 @@
           <!-- <mesh filename="model://blueview_p900_nps_multibeam/meshes/COLLISION-p900.dae" scale="${scale}"/>  -->
           <mesh filename="file://$(find nps_uw_multibeam_sonar)/models/blueview_p900_nps_multibeam/meshes/COLLISION-p900.dae" scale="${scale}"/>
-        </geometry> -->
+        </geometry>
         <pose xyz="0 0 0" rpy="0 0 0"/>
       </collision>
@@ -41,8 +41,10 @@
           <horizontal_fov>1.57079632679</horizontal_fov>
           <image>
-            <width>512</width>
+            <!-- <width>512</width> -->
+            <width>684</width>
             <!-- Set vertical FOV by setting image height -->
             <!-- Approx 2 times the spec sheet (sepc: 20 deg.) -->
-            <height>228</height>
+            <!-- <height>228</height> -->
+            <height>342</height>
             <format>R8G8B8</format>
           </image>
@@ -50,4 +52,5 @@
             <near>0.2</near>            <!-- optimal 2m-60m -->
             <far>${maxDistance + 2}</far>
+            <!-- <far>${maxDistance}</far> -->
           </clip>
           <depth_camera>
@@ -60,5 +63,5 @@
         <plugin filename="libnps_multibeam_sonar_ros_plugin.so" name="${name}_sensor_controller">
           <!-- Sonar properties -->
-          <verticalFOV>20</verticalFOV>
+          <verticalFOV>0</verticalFOV>
           <sonarFreq>900e3</sonarFreq>
           <bandwidth>29.9e3</bandwidth>
